File: MotorDriver.kicad_pcb (KiCad board)
At the start: 8 copper layers, 50 x 50 mm, 108 parts, among them J1 Conn_01x02, J101 USB4105-GF-A, J2 Conn_01x02, J3 Conn_01x02, J4 Conn_01x02, J5 Conn_01x02, J6 Conn_01x02, Q1 BSC040N08NS5, Q2 BSC040N08NS5, Q3 BSC040N08NS5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

Commit message: populate 10k
Parts:
- R7: value 0 -> 10k
- U1, U5, U6: value ~ -> G2026
Changed lines of the file:
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@@
 			)
 		)
-		(property "Value" "~"
+		(property "Value" "G2026"
 			(at 0 3.4 0)
 			(layer "F.Fab")
@@
 			)
 		)
-		(property "Value" "~"
+		(property "Value" "G2026"
 			(at 0 3.4 0)
 			(layer "F.Fab")
@@
 			)
 		)
-		(property "Value" "0"
+		(property "Value" "10k"
 			(at 0 1.17 0)
 			(layer "F.Fab")
@@
 		(sheetname "/")
 		(sheetfile "MotorDriver.kicad_sch")
-		(attr smd dnp)
+		(attr smd)
 		(fp_line
 			(start -0.153641 -0.38)
@@
 			)
 		)
-		(property "Value" "~"
+		(property "Value" "G2026"
 			(at 0 3.4 0)
 			(layer "F.Fab")
@@
 		(fp_text user "*"
 			(at -2.9097 3.6068 90)
-			(unlocked yes)
 			(layer "B.SilkS")
 			(effects
@@
 		(fp_text user "*"
 			(at -2.9097 3.6068 90)
+			(unlocked yes)
 			(layer "B.SilkS")
 			(effects
@@
 			)
 		)
-		(fp_text user "${REFERENCE}"
-			(at 0 0 90)
+		(fp_text user "*"
+			(at -1.5748 2.3749 90)
 			(unlocked yes)
 			(layer "B.Fab")
@@
 			)
 		)
-		(fp_text user "*"
-			(at -1.5748 2.3749 90)
+		(fp_text user "${REFERENCE}"
+			(at 0 0 90)
+			(unlocked yes)
 			(layer "B.Fab")
 			(effects
@@
 		(fp_text user "*"
 			(at -1.5748 2.3749 90)
-			(unlocked yes)
 			(layer "B.Fab")
 			(effects
